File: Lightmeter/Lightmeter.kicad_pcb (KiCad board)
At the start: 2 copper layers, 68.6 x 69.8 mm, 73 parts, among them IC1 FS312F-G, J1 Conn_01x03_Socket, J2 Conn_01x02_Pin, J3 Conn_01x05_Pin, J4 Conn_01x08_Socket, J5 TP4056, P1 USB_C_Plug_USB2.0, Q1 FS8205, SW1 SW_DPDT_x2, U1 RP2040, U2 EC11E1544505, U3 AP2112K-3.3, U4 W25Q32JVSS, U5 MT3608, Y1 Crystal

Commit message: update
Routing:
- net GNDREF: track 0.00 -> 50.8 mm, vias 0 -> 2
- net /LiPo/BAT: track 0.00 -> 27.3 mm, vias 0 -> 2
- net Net-(U5-SW): track 0.00 -> 24.7 mm, vias 0 -> 4
- net Net-(IC1-VCC): track 0.00 -> 21.7 mm
- net Net-(SW1A-C): track 0.00 -> 16.1 mm
- net Net-(U5-FB): track 0.00 -> 16.1 mm, vias 0 -> 2
- net Net-(J5-BAT): track 0.00 -> 15.6 mm
- net /Power/VSYS: track 0.00 -> 7.94 mm
- net Net-(IC1-OD): track 0.00 -> 7.46 mm, vias 0 -> 2
- net +5V: track 15.7 -> 22.8 mm
- net Net-(IC1-CS): track 0.00 -> 4.65 mm
- net Net-(IC1-OC): track 0.00 -> 3.85 mm
- net Net-(D4-K): track 0.00 -> 2.44 mm
- net Net-(J5-PROG2): track 0.00 -> 2.27 mm
- net Net-(D5-K): track 0.00 -> 2.18 mm

Commit message: V2
Parts:
- removed C10, C11, C13, C14, C15, C16, C17, C18, C21, C25, C6, C7, C8: 0.1uF, Capacitor_SMD:C_0603_1608Metric_Pad1.08x0.95mm_HandSolder
- removed C12, C9: 1uF, Capacitor_SMD:C_0603_1608Metric_Pad1.08x0.95mm_HandSolder
- removed C19, C20: 1uF, Capacitor_SMD:C_1206_3216Metric_Pad1.33x1.80mm_HandSolder
- removed C22: 10uF, Capacitor_SMD:C_1206_3216Metric_Pad1.33x1.80mm_HandSolder
- removed C23, C24: 22uF, Capacitor_SMD:C_1206_3216Metric_Pad1.33x1.80mm_HandSolder
- removed D3: SS34, SamacSys_Parts:DIOM7959X262N
- removed D4, D5: LED, LED_SMD:LED_0805_2012Metric_Pad1.15x1.40mm_HandSolder
- removed IC1: FS312F-G, SamacSys_Parts:SOT95P280X145-6N
- removed J5: TP4056, SamacSys_Parts:SOIC127P600X175-9N
- removed L1: 22uH, Inductor_SMD:L_1008_2520Metric
- removed P1: USB_C_Plug_USB2.0, Connector_USB:USB_C_Receptacle_G-Switch_GT-USB-7010ASV
- removed Q1: FS8205, SamacSys_Parts:FS8205
- removed R12, R13: 5.1k 1%, Resistor_SMD:R_0603_1608Metric_Pad0.98x0.95mm_HandSolder
- removed R14, R16: 10k, Resistor_SMD:R_0603_1608Metric_Pad0.98x0.95mm_HandSolder
- removed R15, R19, R20, R21: 1k, Resistor_SMD:R_0603_1608Metric_Pad0.98x0.95mm_HandSolder
- removed R17: 2k, Resistor_SMD:R_0603_1608Metric_Pad0.98x0.95mm_HandSolder
- removed R18: 7.5k, Resistor_SMD:R_0603_1608Metric_Pad0.98x0.95mm_HandSolder
- removed R22, R23, R24: 100, Resistor_SMD:R_0603_1608Metric_Pad0.98x0.95mm_HandSolder
- removed SW1: SW_DPDT_x2, Button_Switch_THT:SW_CuK_JS202011AQN_DPDT_Angled
- removed U3: AP2112K-3.3, Package_TO_SOT_SMD:SOT-23-5_HandSoldering
- removed U4: W25Q32JVSS, Package_SO:SOIC-8_5.23x5.23mm_P1.27mm
- removed U5: MT3608, Package_TO_SOT_SMD:SOT-23-6
- removed Y1: Crystal, Crystal:Crystal_SMD_3225-4Pin_3.2x2.5mm_HandSoldering
- added JP1: Jumper_2_Open, Jumper:SolderJumper-2_P1.3mm_Open_RoundedPad1.0x1.5mm, B.Cu at (172.8, 105.1)
- added JP2: Jumper_2_Open, Jumper:SolderJumper-2_P1.3mm_Open_RoundedPad1.0x1.5mm, B.Cu at (168.9, 105.1)
- added S4: PTS810SJK250SMTRLFS, SamacSys_Parts:PTS810SJG250SMTRLFS, B.Cu at (161.3, 93.8)
- C1, C2: value 27pF -> 0.1uF; footprint Capacitor_SMD:C_0603_1608Metric_Pad1.08x0.95mm_HandSolder -> Capacitor_SMD:C_1206_3216Metric_Pad1.33x1.80mm_HandSolder
- C3, C4, C5: footprint Capacitor_SMD:C_0603_1608Metric_Pad1.08x0.95mm_HandSolder -> Capacitor_SMD:C_1206_3216Metric_Pad1.33x1.80mm_HandSolder
- D1: footprint LED_SMD:LED_0805_2012Metric_Pad1.15x1.40mm_HandSolder -> LED_SMD:LED_1206_3216Metric_Pad1.42x1.75mm_HandSolder
- D2: value MBR120LSFT1G -> LED; footprint SamacSys_Parts:SODFL3616X98N -> LED_SMD:LED_1206_3216Metric_Pad1.42x1.75mm_HandSolder
- J1: value Conn_01x03_Socket -> USB_C_Receptacle_USB2.0; footprint Connector_PinHeader_2.54mm:PinHeader_1x03_P2.54mm_Vertical -> Connector_USB:USB_C_Receptacle_GCT_USB4105-xx-A_16P_TopMnt_Horizontal
- J2: value Conn_01x02_Pin -> Conn_01x02_Socket; footprint Connector_PinHeader_2.54mm:PinHeader_1x02_P2.54mm_Vertical -> Connector_JST:JST_PH_S2B-PH-SM4-TB_1x02-1MP_P2.00mm_Horizontal; moved to B.Cu
- R1: value DNP -> 5.1k; footprint Resistor_SMD:R_0603_1608Metric_Pad0.98x0.95mm_HandSolder -> Resistor_SMD:R_1206_3216Metric_Pad1.30x1.75mm_HandSolder
- R10, R11, R7, R8, R9: footprint Resistor_SMD:R_0603_1608Metric_Pad0.98x0.95mm_HandSolder -> Resistor_SMD:R_1206_3216Metric_Pad1.30x1.75mm_HandSolder
- R2: value 1k -> 5.1k; footprint Resistor_SMD:R_0603_1608Metric_Pad0.98x0.95mm_HandSolder -> Resistor_SMD:R_1206_3216Metric_Pad1.30x1.75mm_HandSolder
- R3: value 1k -> 100k; footprint Resistor_SMD:R_0603_1608Metric_Pad0.98x0.95mm_HandSolder -> Resistor_SMD:R_1206_3216Metric_Pad1.30x1.75mm_HandSolder
- R4: value 27 -> 100k; footprint Resistor_SMD:R_0603_1608Metric_Pad0.98x0.95mm_HandSolder -> Resistor_SMD:R_1206_3216Metric_Pad1.30x1.75mm_HandSolder
- R5: value 27 -> 1k; footprint Resistor_SMD:R_0603_1608Metric_Pad0.98x0.95mm_HandSolder -> Resistor_SMD:R_1206_3216Metric_Pad1.30x1.75mm_HandSolder
- R6: value 10k -> 1k; footprint Resistor_SMD:R_0603_1608Metric_Pad0.98x0.95mm_HandSolder -> Resistor_SMD:R_1206_3216Metric_Pad1.30x1.75mm_HandSolder
- S3: moved to B.Cu
- U1: value RP2040 -> RP2040_Stamp; footprint Package_DFN_QFN:QFN-56-1EP_7x7mm_P0.4mm_EP3.2x3.2mm -> RP2040_Stamp:RP2040_Stamp_SMD
- moved C3 90.8 mm to (157.6, 129.1)
- moved C4 86.9 mm to (168.9, 106.0), turned to 90 degrees
- moved J1 81.8 mm to (141.6, 126.4)
- moved C5 81.2 mm to (150.7, 129.1)
- moved J2 74.0 mm to (133.3, 114.9), turned to -90 degrees
- moved C1 68.1 mm to (169.5, 128.9), turned to -90 degrees
- moved R3 64.5 mm to (130.8, 113.5)
- moved D1 60.9 mm to (172.8, 94.5), turned to -90 degrees
- moved R1 58.7 mm to (139.6, 118.4), turned to 90 degrees
- moved J4 58.5 mm to (130.2, 89.5)
- moved R2 54.0 mm to (143.4, 118.4), turned to 90 degrees
- moved C2 52.9 mm to (173.4, 128.9), turned to -90 degrees
- moved R4 51.4 mm to (130.8, 116.8)
- moved S1 47.2 mm to (157.7, 123.2), turned to -90 degrees
- moved R5 46.4 mm to (172.9, 100.3), turned to -90 degrees
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Connections:
- C1 pad 1: /XIN -> /EN_CLK
- C2 pad 1: Net-(C2-Pad1) -> /EN_DT
- C3 pad 1: +3.3V -> Net-(C3-Pad1)
- C4 pad 1: +3.3V -> /EN_SW
- C5 pad 1: +3.3V -> Net-(C5-Pad1)
- D2 pad 1: /Power/VSYS -> /LED_USR
- D2 pad 2: +5V -> Net-(D2-A)
- J2 pad 1: GNDREF -> +BATT
- J2 pad 2: /RUN -> GNDREF
- R1 pad 1: /XIN -> Net-(J1-CC1)
- R1 pad 2: /XOUT -> GNDREF
- R10 pad 1: /MEAS -> +3.3V
- R10 pad 2: +3.3V -> /MEAS
- R2 pad 1: Net-(C2-Pad1) -> Net-(J1-CC2)
- R2 pad 2: /XOUT -> GNDREF
- R3 pad 1: /GPIO25 -> +BATT
- R3 pad 2: Net-(D1-A) -> /VDIV
- R4 pad 1: /USB_P -> /VDIV
- R4 pad 2: Net-(U1-USB_DP) -> GNDREF
- R5 pad 1: Net-(U1-USB_DM) -> Net-(JP1-A)
- R5 pad 2: /USB_N -> Net-(D1-A)
- R6 pad 1: /RUN -> Net-(JP2-A)
- R6 pad 2: +3.3V -> Net-(D2-A)
- R8 pad 1: /ISO -> +3.3V
- R8 pad 2: +3.3V -> /ISO
- S1 pad 3: Net-(C16-Pad1) -> Net-(C3-Pad1)
- S1 pad 4: Net-(C16-Pad1) -> Net-(C3-Pad1)
- S2 pad 3: Net-(C18-Pad1) -> Net-(C5-Pad1)
- S2 pad 4: Net-(C18-Pad1) -> Net-(C5-Pad1)
- S3 pad 1: /Flash/USB_BOOT -> /BOOTSEL
- S3 pad 2: /Flash/USB_BOOT -> /BOOTSEL
- U1 pad 1: +3.3V -> unconnected-(U1-GPIO0-Pad1)
- U1 pad 10: +3.3V -> /EN_SW
- U1 pad 11: /EN_SW -> unconnected-(U1-GPIO10-Pad11)
- U1 pad 17: unconnected-(U1-GPIO14-Pad17) -> /MEAS
- U1 pad 18: /MEAS -> unconnected-(U1-GPIO17-Pad18)
- U1 pad 19: GNDREF -> /SCREEN_CS
- U1 pad 20: /XIN -> /SCREEN_SCK
- U1 pad 21: /XOUT -> /SCREEN_MOSI
- U1 pad 22: +3.3V -> /SCREEN_DC
- U1 pad 23: /+1.1V -> /SCREEN_RST
- U1 pad 24: /SWCLK -> /ISO
- U1 pad 25: /SWDIO -> /LED_USR
- U1 pad 26: /RUN -> unconnected-(U1-GPIO25-Pad26)
- U1 pad 27: unconnected-(U1-GPIO16-Pad27) -> /VDIV
- U1 pad 28: /SCREEN_CS -> unconnected-(U1-GPIO27-Pad28)
- U1 pad 29: /SCREEN_SCK -> unconnected-(U1-GPIO28-Pad29)
- U1 pad 30: /SCREEN_MOSI -> unconnected-(U1-GPIO29-Pad30)
- U1 pad 31: /SCREEN_DC -> GNDREF
- U1 pad 32: /SCREEN_RST -> +BATT
- U1 pad 33: +3.3V -> +5V
- U1 pad 34: /ISO -> +3.3V
- U1 pad 35: unconnected-(U1-GPIO23-Pad35) -> /USB_D-
- U1 pad 36: unconnected-(U1-GPIO24-Pad36) -> /USB_D+
- U1 pad 37: /GPIO25 -> unconnected-(U1-SWDIO-Pad37)
- U1 pad 39: unconnected-(U1-GPIO27_ADC1-Pad39) -> /~{RESET}
- U1 pad 4: /L_SDA -> unconnected-(U1-GPIO3-Pad4)
- U1 pad 40: unconnected-(U1-GPIO28_ADC2-Pad40) -> /BOOTSEL
- U1 pad 5: /L_SCL -> /L_SDA
- U1 pad 6: unconnected-(U1-GPIO4-Pad6) -> /L_SCL
Routing:
- net GNDREF: track 50.8 -> 0.00 mm, vias 2 -> 0
- net /LiPo/BAT: track 27.3 -> 0.00 mm, vias 2 -> 0
- net Net-(U5-SW): track 24.7 -> 0.00 mm, vias 4 -> 0
- net +5V: track 22.8 -> 0.00 mm, vias 2 -> 0
- net Net-(IC1-VCC): track 21.7 -> 0.00 mm
- net Net-(SW1A-C): track 16.1 -> 0.00 mm
- net Net-(U5-FB): track 16.1 -> 0.00 mm, vias 2 -> 0
- net Net-(J5-BAT): track 15.6 -> 0.00 mm
- net /Power/VSYS: track 7.94 -> 0.00 mm
- net Net-(IC1-OD): track 7.46 -> 0.00 mm, vias 2 -> 0
- net Net-(U1-VREG_IN): track 5.25 -> 0.00 mm
- net Net-(IC1-CS): track 4.65 -> 0.00 mm
- net Net-(U1-VREG_VOUT): track 4.04 -> 0.00 mm
- net Net-(P1-VCONN): track 3.88 -> 0.00 mm
- net Net-(IC1-OC): track 3.85 -> 0.00 mm
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- removed copper zone on B.Cu, net +3.3V
- removed copper zone on F.Cu, net +5V
- removed copper zone on F.Cu, net GNDREF
Other:
- board size 68.6 x 69.8 mm -> 53.3 x 52.7 mm
