File: Lightmeter/Lightmeter.kicad_sch (KiCad schematic)
At the start: 39 parts, among them J1 Conn_01x03_Socket, J2 Conn_01x02_Pin, J3 Conn_01x05_Pin, J4 Conn_01x08_Socket, U1 RP2040, U2 EC11E1544505, Y1 Crystal

Commit message: V2
Parts:
- removed C? (x14): 0.1uF, Capacitor_SMD:C_0603_1608Metric_Pad1.08x0.95mm_HandSolder, symbol Device:C
- removed C? (x2): 27pF, Capacitor_SMD:C_0603_1608Metric_Pad1.08x0.95mm_HandSolder, symbol Device:C
- removed C? (x2): 1uF, Capacitor_SMD:C_0603_1608Metric_Pad1.08x0.95mm_HandSolder, symbol Device:C
- removed J1: Conn_01x03_Socket, Connector_PinHeader_2.54mm:PinHeader_1x03_P2.54mm_Vertical, symbol Connector:Conn_01x03_Socket
- removed J2: Conn_01x02_Pin, Connector_PinHeader_2.54mm:PinHeader_1x02_P2.54mm_Vertical, symbol Connector:Conn_01x02_Pin
- removed S? (x2): PTS810SJK250SMTRLFS, PTS810SJG250SMTRLFS, symbol SamacSys_Parts:PTS810SJK250SMTRLFS
- removed U1: RP2040, Package_DFN_QFN:QFN-56-1EP_7x7mm_P0.4mm_EP3.2x3.2mm, symbol MCU_RaspberryPi:RP2040
- removed Y1: Crystal, Crystal:Crystal_SMD_3225-4Pin_3.2x2.5mm_HandSoldering, symbol Device:Crystal
- added C? (x5): 0.1uF, Capacitor_SMD:C_1206_3216Metric_Pad1.33x1.80mm_HandSolder, symbol Device:C
- added D2: LED, LED_SMD:LED_1206_3216Metric_Pad1.42x1.75mm_HandSolder, symbol Device:LED
- added J1: USB_C_Receptacle_USB2.0, Connector_USB:USB_C_Receptacle_GCT_USB4105-xx-A_16P_TopMnt_Horizontal, symbol Connector:USB_C_Receptacle_USB2.0
- added J2: Conn_01x02_Socket, Connector_JST:JST_PH_S2B-PH-SM4-TB_1x02-1MP_P2.00mm_Horizontal, symbol Connector:Conn_01x02_Socket
- added JP1, JP2: Jumper_2_Open, Jumper:SolderJumper-2_P1.3mm_Open_RoundedPad1.0x1.5mm, symbol Jumper:Jumper_2_Open
- added S3 (x2), S? (x2): PTS810SJK250SMTRLFS, PTS810SJG250SMTRLFS, symbol SamacSys_Parts:PTS810SJK250SMTRLFS
- added U1: RP2040_Stamp, RP2040_Stamp:RP2040_Stamp_SMD, symbol RP2040_Stamp:RP2040_Stamp
- D1: footprint LED_SMD:LED_0805_2012Metric_Pad1.15x1.40mm_HandSolder -> LED_SMD:LED_1206_3216Metric_Pad1.42x1.75mm_HandSolder
- R1: value DNP -> 5.1k; footprint Resistor_SMD:R_0603_1608Metric_Pad0.98x0.95mm_HandSolder -> Resistor_SMD:R_1206_3216Metric_Pad1.30x1.75mm_HandSolder
- R10, R11, R7, R8, R9: footprint Resistor_SMD:R_0603_1608Metric_Pad0.98x0.95mm_HandSolder -> Resistor_SMD:R_1206_3216Metric_Pad1.30x1.75mm_HandSolder
- R2: value 1k -> 5.1k; footprint Resistor_SMD:R_0603_1608Metric_Pad0.98x0.95mm_HandSolder -> Resistor_SMD:R_1206_3216Metric_Pad1.30x1.75mm_HandSolder
- R3: value 1k -> 100k; footprint Resistor_SMD:R_0603_1608Metric_Pad0.98x0.95mm_HandSolder -> Resistor_SMD:R_1206_3216Metric_Pad1.30x1.75mm_HandSolder
- R4: value 27 -> 100k; footprint Resistor_SMD:R_0603_1608Metric_Pad0.98x0.95mm_HandSolder -> Resistor_SMD:R_1206_3216Metric_Pad1.30x1.75mm_HandSolder
- R5: value 27 -> 1k; footprint Resistor_SMD:R_0603_1608Metric_Pad0.98x0.95mm_HandSolder -> Resistor_SMD:R_1206_3216Metric_Pad1.30x1.75mm_HandSolder
- R6: value 10k -> 1k; footprint Resistor_SMD:R_0603_1608Metric_Pad0.98x0.95mm_HandSolder -> Resistor_SMD:R_1206_3216Metric_Pad1.30x1.75mm_HandSolder
Connections:
- net USB_N is gone; now on an unnamed net: R5.2
- net XOUT is gone; now on net GNDREF: R1.2, R2.2
- net +3.3V: now also R10.1, R8.1, JP1.2 (B), JP2.2 (B), U1.34 (3.3V); no longer R10.2, R6.2, R8.2
- net EN_CLK: now also C?.1, U1.8 (GPIO7)
- net EN_DT: now also C?.1, U1.9 (GPIO8)
- net EN_SW: now also C?.1, U1.10 (GPIO9)
- net GNDREF: now also R4.2, C?.2, C?.2, C?.2, C?.2, C?.2, J1.A1 (GND), J1.A12 (GND), J1.B1 (GND), J1.B12 (GND), J1.S1 (SHIELD), J2.2 (Pin_2), S3.3, S3.3, S3.4, S3.4, U1.31 (GND)
- net ISO: now also R8.2, S?.1, S?.2, U1.24 (GPIO23); no longer R8.1
- net L_SCL: now also U1.6 (GPIO5)
- net L_SDA: now also U1.5 (GPIO4)
- net MEAS: now also R10.2, S?.1, S?.2, U1.17 (GPIO16); no longer R10.1
- net SCREEN_CS: now also U1.19 (GPIO18)
- net SCREEN_DC: now also U1.22 (GPIO21)
- net SCREEN_MOSI: now also U1.21 (GPIO20)
- net SCREEN_RST: now also U1.23 (GPIO22)
- net SCREEN_SCK: now also U1.20 (GPIO19)
- net at R2.1: now also J1.B5 (CC2)
- net at D1.2 (A): no longer R3.2
- net at R5.1: now also JP1.1 (A)
- net GPIO25 renamed +BATT
- net +BATT: now also J2.1 (Pin_1), U1.32 (VBAT)
- net RUN: no longer names the net of R6.1
- net RUN: now also JP2.1 (A)
- net USB_P renamed VDIV
- net VDIV: now also R3.2, U1.27 (GPIO26)
- net XIN: no longer names the net of R1.1
- net XIN: now also J1.A5 (CC1)
- new net: D2.2 (A), R6.2
- new net: C?.1, S?.3, S?.4 (x2)
- new net +5V: U1.33 (5V)
- new net BOOTSEL: S3.1, S3.2, U1.40 (BOOTSEL)
- new net LED_USR: D2.1 (K), U1.25 (GPIO24)
- new net USB_D+: J1.A6 (D+), J1.B6 (D+), U1.36 (USB_D+)
- new net USB_D-: J1.A7 (D-), J1.B7 (D-), U1.35 (USB_D-)
- new net VBUS: J1.A4 (VBUS), J1.A9 (VBUS), J1.B4 (VBUS), J1.B9 (VBUS)
- new net ~{RESET}: S3.1, S3.2, U1.39 (~{RESET})
- no-connect marks 19 -> 4
Other:
- removed sheet Flash
- removed sheet LiPo
- removed sheet Power
- note added: "3.3v power indictor and user adressable led"
- note added: "Battery connector and voltage measurement"
- note added: "Bootselect and reset buttons"
- note added: "USB-C connector with power selector resistors"
- note removed: "Clock"
- note removed: "Debug ports"
- note removed: "Decoupling capacitors"
- note removed: "General purpose LED"
- note removed: "Place close to ADC_AVDD"
- note removed: "Place each close to a DVDD pin"
- note removed: "Place each close to a IOVDD pin"
- title: (none) -> Lightmeter for analog photography
