File: Lightmeter/versions/v1/Lightmeter.kicad_pcb (KiCad board)
At the start: 2 copper layers, 68.6 x 69.8 mm, 73 parts, among them IC1 FS312F-G, J1 Conn_01x03_Socket, J2 Conn_01x02_Pin, J3 Conn_01x05_Pin, J4 Conn_01x08_Socket, J5 TP4056, P1 USB_C_Plug_USB2.0, Q1 FS8205, SW1 SW_DPDT_x2, U1 RP2040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

Commit message: Update
Parts:
- added R25: 10k, Resistor_SMD:R_1206_3216Metric_Pad1.30x1.75mm_HandSolder, F.Cu at (95.6, 51.4)
Changed lines of the file:
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@@
   (net 80 "+5V")
   (net 81 "Net-(J5-PROG2)")
+  (net 82 "unconnected-(R25-Pad1)")
+  (net 83 "unconnected-(R25-Pad2)")
   (footprint "Capacitor_SMD:C_0603_1608Metric_Pad1.08x0.95mm_HandSolder" (layer "F.Cu")
     (at 129.032 110.49 90)
@@
     (property "ki_description" "One Cell Lithium-ion/Polymer Battery Protection IC")
     (attr smd)
-    (fp_text reference "IC1" (at 0 0) (layer "F.SilkS")
+    (fp_text reference "IC1" (at 0 3.302) (layer "F.SilkS")
         (effects (font (size 1.27 1.27) (thickness 0.254)))
     )
@@
     )
   )
+  (footprint "Resistor_SMD:R_1206_3216Metric_Pad1.30x1.75mm_HandSolder" (layer "F.Cu")
+    (at 95.605 51.435)
+    (descr "Resistor SMD 1206 (3216 Metric), square (rectangular) end terminal, IPC_7351 nominal with elongated pad for handsoldering. (Body size source: IPC-SM-782 page 72, https://www.pcb-3d.com/wordpress/wp-content/uploads/ipc-sm-782a_amendment_1_and_2.pdf), generated with kicad-footprint-generator")
+    (tags "resistor handsolder")
+    (property "Sheetfile" "Lightmeter.kicad_sch")
+    (property "Sheetname" "")
+    (property "ki_description" "Resistor")
+    (property "ki_keywords" "R res resistor")
+    (attr smd)
+    (fp_text reference "R25" (at 0 -1.82) (layer "F.SilkS")
+        (effects (font (size 1 1) (thickness 0.15)))
+    )
+    (fp_text value "10k" (at 0 1.82) (layer "F.Fab")
+        (effects (font (size 1 1) (thickness 0.15)))
+    )
+    (fp_text user "${REFERENCE}" (at 0 0) (layer "F.Fab")
+        (effects (font (size 0.8 0.8) (thickness 0.12)))
+    )
+    (fp_line (start -0.727064 -0.91) (end 0.727064 -0.91)
+      (stroke (width 0.12) (type solid)) (layer "F.SilkS"))
+    (fp_line (start -0.727064 0.91) (end 0.727064 0.91)
+      (stroke (width 0.12) (type solid)) (layer "F.SilkS"))
+    (fp_line (start -2.45 -1.12) (end 2.45 -1.12)
+      (stroke (width 0.05) (type solid)) (layer "F.CrtYd"))
+    (fp_line (start -2.45 1.12) (end -2.45 -1.12)
+      (stroke (width 0.05) (type solid)) (layer "F.CrtYd"))
+    (fp_line (start 2.45 -1.12) (end 2.45 1.12)
+      (stroke (width 0.05) (type solid)) (layer "F.CrtYd"))
+    (fp_line (start 2.45 1.12) (end -2.45 1.12)
+      (stroke (width 0.05) (type solid)) (layer "F.CrtYd"))
+    (fp_line (start -1.6 -0.8) (end 1.6 -0.8)
+      (stroke (width 0.1) (type solid)) (layer "F.Fab"))
+    (fp_line (start -1.6 0.8) (end -1.6 -0.8)
+      (stroke (width 0.1) (type solid)) (layer "F.Fab"))
+    (fp_line (start 1.6 -0.8) (end 1.6 0.8)
+      (stroke (width 0.1) (type solid)) (layer "F.Fab"))
+    (fp_line (start 1.6 0.8) (end -1.6 0.8)
+      (stroke (width 0.1) (type solid)) (layer "F.Fab"))
+    (pad "1" smd roundrect (at -1.55 0) (size 1.3 1.75) (layers "F.Cu" "F.Paste" "F.Mask") (roundrect_rratio 0.192308)
+      (net 82 "unconnected-(R25-Pad1)") (pintype "passive"))
+    (pad "2" smd roundrect (at 1.55 0) (size 1.3 1.75) (layers "F.Cu" "F.Paste" "F.Mask") (roundrect_rratio 0.192308)
+      (net 83 "unconnected-(R25-Pad2)") (pintype "passive"))
+    (model "${KICAD6_3DMODEL_DIR}/Resistor_SMD.3dshapes/R_1206_3216Metric.wrl"
+      (offset (xyz 0 0 0))
+      (scale (xyz 1 1 1))
+      (rotate (xyz 0 0 0))
+    )
+  )
   (footprint "SamacSys_Parts:SODFL3616X98N" (layer "F.Cu")
     (at 153.416 102.87 -90)
@@
     (property "ki_description" "TAIWAN SEMICONDUCTOR - SS34 - DIODE, SCHOTTKY, 3A, 40V")
     (attr smd)
-    (fp_text reference "D3" (at 0 0) (layer "F.SilkS")
+    (fp_text reference "D3" (at 0 0 180) (layer "F.SilkS")
         (effects (font (size 1.27 1.27) (thickness 0.254)))
     )
-    (fp_text value "SS34" (at 0 0) (layer "F.SilkS") hide
+    (fp_text value "SS34" (at 0 0 180) (layer "F.SilkS") hide
         (effects (font (size 1.27 1.27) (thickness 0.254)))
     )
-    (fp_text user "${REFERENCE}" (at 0 0) (layer "F.Fab")
+    (fp_text user "${REFERENCE}" (at 0 0 180) (layer "F.Fab")
         (effects (font (size 1.27 1.27) (thickness 0.254)))
     )
